Commit message: taller 11 terminado

File: taller11/URDF/bot.urdf (robot description, URDF)
Before this commit: robot Pioneer_p3dx, 5 links, 4 joints
Links:
- removed link base_link
- added link base_link_gt, mass 16.0; collision box size=0.005000 0.030000 0.045000; collision box size=0.005000 0.030000 0.045000
Joints:
- joint Pioneer_p3dx_caster_freeJoint1: parent base_link -> base_link_gt
- joint Pioneer_p3dx_leftMotor: parent base_link -> base_link_gt
- joint Pioneer_p3dx_rightMotor: parent base_link -> base_link_gt
